File: kicad_files/APA102C_8x8_Matrix.sch (KiCad schematic (older format))
At the start: 0 parts

Commit message: a days work submitted
Other:
- note removed: "03-13-2015"
- note removed: "APA102C 8x8 Matrix"
Changed lines of the file:
@@
 LIBS:contrib
 LIBS:valves
-EELAYER 25 0
+LIBS:ab2_7segment
+LIBS:ab2_audio
+LIBS:ab2_buffer
+LIBS:ab2_capacitor
+LIBS:ab2_connectivity
+LIBS:ab2_dac
+LIBS:ab2_diode
+LIBS:ab2_gpio_expansion
+LIBS:ab2_header
+LIBS:ab2_idc
+LIBS:ab2_inductor
+LIBS:ab2_input_devices
+LIBS:ab2_jumper
+LIBS:ab2_lcd
+LIBS:ab2_led
+LIBS:ab2_opamp
+LIBS:ab2_pot
+LIBS:ab2_power
+LIBS:ab2_regulator
+LIBS:ab2_relay
+LIBS:ab2_resistor
+LIBS:ab2_sensor
+LIBS:ab2_stepper
+LIBS:ab2_supply
+LIBS:ab2_terminal_block
+LIBS:ab2_test
+LIBS:ab2_transistor
+LIBS:ab2_uC
+LIBS:ab2_usb
+LIBS:ab2_xtal
+LIBS:APA102C_8x8_Matrix-cache
+EELAYER 27 0
 EELAYER END
-$Descr A4 11693 8268
+$Descr USLegal 14000 8500
 encoding utf-8
 Sheet 1 1
-Title ""
-Date ""
-Rev ""
-Comp ""
+Title "APA102C_8x8_Matrix"
+Date "14 mar 2015"
+Rev "1.0"
+Comp "ProckNation.com"
 Comment1 ""
 Comment2 ""
@@
 Comment4 ""
 $EndDescr
-Text Notes 8150 7650 0    60   ~ 0
-03-13-2015
-Text Notes 7350 7500 0    67   ~ 0
-APA102C 8x8 Matrix
 $EndSCHEMATC
